File: kicad/duet_micro_tool.sch (KiCad schematic (older format))
At the start: 41 parts, among them J1 Conn_01x04_Male, J2 Conn_01x05_Male, U1 ATSAMC21G18A-AUT, U2 L78M05ABDT-TR, U3 XC6206P332MR, U4 LIS3DH, U5 MCP2542FDxMF, X1 25Mhz

Commit message: Work in progress
Parts:
- added C?: 10n, symbol Device:C
- added D?: GREEN, symbol duet_micro_tool:LED
- added R? (x3): 4k7, symbol Device:R_US
- added R?: 60k, symbol Device:R_US
- added R?: 1k, symbol Device:R_US
- D2: value BLUE -> RED
- D3: value GREEN -> RED
- R1: value 22k -> 1k
- R2: value 1k -> 10k
- R6: value 10k -> 1k
Connections:
- net 3.3V: now also D2.2 (A), U1.12 (PA07), D?.2 (A), R?.2, R?.2
- net GND: now also U1.11 (PA06), U1.7 (PB08), C?.1, R?.1; no longer D2.1 (K)
- net I2C_SDA: now also R?.1
- net POWER: no longer R6.2
- net SWDCLK: now also R6.1
- net SWDIO: now also R?.1
- net VIN+: now also R?.2
- net VIN_MON: now reaches U1.13 (PA08)
- net VIN_MON: now also C?.2, R?.1, R?.2
- new net: D2.1 (K), R6.2
- new net: D?.1 (K), R?.2
- no-connect marks 27 -> 23
Other:
- note added: "ACT"
- note added: "POWER"
- note added: "STATUS"
- note added: "TODO: Add pull up/down for unused inputs."
- note added: "TODO: Does accelerator's int1 need pull up?"
- note added: "TODO: Verify 5V LDO max power"
- note added: "VIN 12VDC/24VDC"
- note removed: "8VDC to 24VDC"
- note removed: "TODO: Ok to leave all MPU inputs floating?"
- note removed: "TODO: VMON signals needed?"
- note removed: "TODO: Verify 5V LDO power"
- moved on the sheet: D2, D3, J2, R6, R7

Commit message: Work in progress
Parts:
- added C?: 100n, symbol Device:C
Connections:
- net 3.3V: now also U1.36 (VDDIO), C?.2
- net GND: now also U1.35 (GND), C?.1
Changed lines of the file:
@@
 Text Notes 7325 5550 0    50   ~ 0
 ACT
+$Comp
+L Device:C C?
+U 1 1 624C7381
+P 4700 5950
+F 0 "C?" H 4550 5850 50  0000 L CNN
+F 1 "100n" H 4500 6050 50  0000 L CNN
+F 2 "" H 4738 5800 50  0001 C CNN
+F 3 "~" H 4700 5950 50  0001 C CNN
+F 4 "C307331" H 4700 5950 50  0001 C CNN "LCSC Part Number"
+	1    4700 5950
+	-1   0    0    1
+$EndComp
+Wire Wire Line
+	4500 6150 4700 6150
+Wire Wire Line
+	4500 5750 4700 5750
+Wire Wire Line
+	4700 5750 4700 5800
+Text GLabel 4900 5750 2    50   Input ~ 0
+3.3V
+Wire Wire Line
+	4700 5750 4900 5750
+Connection ~ 4700 5750
+$Comp
+L power:GND #PWR?
+U 1 1 6250AF69
+P 4700 6175
+F 0 "#PWR?" H 4700 5925 50  0001 C CNN
+F 1 "GND" H 4705 6002 50  0001 C CNN
+F 2 "" H 4700 6175 50  0001 C CNN
+F 3 "" H 4700 6175 50  0001 C CNN
+	1    4700 6175
+	1    0    0    -1
+$EndComp
+Wire Wire Line
+	4700 6100 4700 6150
+Connection ~ 4700 6150
+Wire Wire Line
+	4700 6150 4700 6175
 $EndSCHEMATC
