File: kicad/duet_micro_tool.sch (KiCad schematic (older format))
At the start: 49 parts, among them J1 Conn_01x04_Male, J2 Conn_01x05_Male, U1 ATSAMC21G18A-AUT, U2 L78M05ABDT-TR, U3 XC6206P332MR, U4 LIS3DH, U5 MCP2542FDxMF, X1 25Mhz

Commit message: Work in progress
Connections:
- net 3.3V: now also U1.36 (VDDIO)
Other:
- moved on the sheet: C11, C?, R4
Changed lines of the file:
@@
 3.3V
 Wire Wire Line
-	4650 6500 4650 6400
-Wire Wire Line
-	4900 6400 4900 6500
-Wire Wire Line
-	4650 6800 4650 6900
-Wire Wire Line
-	4900 6900 4900 6800
+	4650 6550 4650 6500
+Wire Wire Line
+	4900 6500 4900 6550
+Wire Wire Line
+	4650 6850 4650 6900
+Wire Wire Line
+	4900 6900 4900 6850
 Wire Wire Line
 	4500 6900 4650 6900
@@
 Wire Wire Line
 	4900 6900 5000 6900
-Text GLabel 5100 6400 2    50   Input ~ 0
+Text GLabel 5125 6500 2    50   Input ~ 0
 3.3V
 $Comp
@@
 L Device:C C11
 U 1 1 61792C11
-P 4900 6650
-F 0 "C11" H 5015 6696 50  0000 L CNN
-F 1 "2n2" H 5015 6605 50  0000 L CNN
-F 2 "" H 4938 6500 50  0001 C CNN
-F 3 "~" H 4900 6650 50  0001 C CNN
-	1    4900 6650
+P 4900 6700
+F 0 "C11" H 5015 6746 50  0000 L CNN
+F 1 "2n2" H 5015 6655 50  0000 L CNN
+F 2 "" H 4938 6550 50  0001 C CNN
+F 3 "~" H 4900 6700 50  0001 C CNN
+	1    4900 6700
 	1    0    0    -1
 $EndComp
@@
 L Device:R_US R4
 U 1 1 61799B13
-P 4650 6650
-F 0 "R4" H 4800 6600 50  0000 R CNN
-F 1 "10K" H 4850 6700 50  0000 R CNN
-F 2 "" V 4690 6640 50  0001 C CNN
-F 3 "~" H 4650 6650 50  0001 C CNN
-	1    4650 6650
+P 4650 6700
+F 0 "R4" H 4800 6650 50  0000 R CNN
+F 1 "10K" H 4850 6750 50  0000 R CNN
+F 2 "" V 4690 6690 50  0001 C CNN
+F 3 "~" H 4650 6700 50  0001 C CNN
+	1    4650 6700
 	-1   0    0    1
 $EndComp
@@
 	5300 6900 5400 6900
 Wire Wire Line
-	4900 6400 5100 6400
-Wire Wire Line
-	4650 6400 4900 6400
+	4900 6500 5125 6500
+Wire Wire Line
+	4650 6500 4900 6500
 Text GLabel 2300 4500 0    50   Input ~ 0
 3.3V
@@
 	1    0    0    -1
 $EndComp
-Connection ~ 4900 6400
+Connection ~ 4900 6500
 $Comp
 L Jumper:SolderJumper_2_Open JP1
@@
 L Device:C C?
 U 1 1 624C7381
-P 4700 5950
-F 0 "C?" H 4550 5850 50  0000 L CNN
-F 1 "100n" H 4500 6050 50  0000 L CNN
-F 2 "" H 4738 5800 50  0001 C CNN
-F 3 "~" H 4700 5950 50  0001 C CNN
-F 4 "C307331" H 4700 5950 50  0001 C CNN "LCSC Part Number"
-	1    4700 5950
-	-1   0    0    1
-$EndComp
-Wire Wire Line
-	4500 6150 4700 6150
-Wire Wire Line
-	4500 5750 4700 5750
-Wire Wire Line
-	4700 5750 4700 5800
-Text GLabel 4900 5750 2    50   Input ~ 0
+P 4650 6100
+F 0 "C?" H 4500 6000 50  0000 L CNN
+F 1 "100n" H 4450 6200 50  0000 L CNN
+F 2 "" H 4688 5950 50  0001 C CNN
+F 3 "~" H 4650 6100 50  0001 C CNN
+F 4 "C307331" H 4650 6100 50  0001 C CNN "LCSC Part Number"
+	1    4650 6100
+	-1   0    0    1
+$EndComp
+Wire Wire Line
+	4500 5900 4650 5900
+Wire Wire Line
+	4650 5900 4650 5950
+Text GLabel 4875 5900 2    50   Input ~ 0
 3.3V
 Wire Wire Line
-	4700 5750 4900 5750
-Connection ~ 4700 5750
+	4650 5900 4875 5900
+Connection ~ 4650 5900
 $Comp
 L power:GND #PWR?
 U 1 1 6250AF69
-P 4700 6175
-F 0 "#PWR?" H 4700 5925 50  0001 C CNN
-F 1 "GND" H 4705 6002 50  0001 C CNN
-F 2 "" H 4700 6175 50  0001 C CNN
-F 3 "" H 4700 6175 50  0001 C CNN
-	1    4700 6175
-	1    0    0    -1
-$EndComp
-Wire Wire Line
-	4700 6100 4700 6150
-Connection ~ 4700 6150
-Wire Wire Line
-	4700 6150 4700 6175
+P 4650 6275
+F 0 "#PWR?" H 4650 6025 50  0001 C CNN
+F 1 "GND" H 4655 6102 50  0001 C CNN
+F 2 "" H 4650 6275 50  0001 C CNN
+F 3 "" H 4650 6275 50  0001 C CNN
+	1    4650 6275
+	1    0    0    -1
+$EndComp
+$Comp
+L power:GND #PWR?
+U 1 1 61C91224
+P 3650 7600
+F 0 "#PWR?" H 3650 7350 50  0001 C CNN
+F 1 "GND" H 3655 7427 50  0001 C CNN
+F 2 "" H 3650 7600 50  0001 C CNN
+F 3 "" H 3650 7600 50  0001 C CNN
+	1    3650 7600
+	1    0    0    -1
+$EndComp
+Wire Wire Line
+	3650 7600 3650 7550
+Wire Wire Line
+	4650 6250 4650 6275
 $EndSCHEMATC

Commit message: Work in progress.
Connections:
- net GND: now also U1.18 (GND), U1.35 (GND), U1.42 (GND), U1.EPAD
Changed lines of the file:
@@
 L power:GND #PWR010
 U 1 1 61783726
-P 3350 7600
-F 0 "#PWR010" H 3350 7350 50  0001 C CNN
-F 1 "GND" H 3355 7427 50  0001 C CNN
-F 2 "" H 3350 7600 50  0001 C CNN
-F 3 "" H 3350 7600 50  0001 C CNN
-	1    3350 7600
+P 3400 7600
+F 0 "#PWR010" H 3400 7350 50  0001 C CNN
+F 1 "GND" H 3405 7427 50  0001 C CNN
+F 2 "" H 3400 7600 50  0001 C CNN
+F 3 "" H 3400 7600 50  0001 C CNN
+	1    3400 7600
 	1    0    0    -1
 $EndComp
@@
 L power:GND #PWR011
 U 1 1 617838A2
-P 3500 7600
-F 0 "#PWR011" H 3500 7350 50  0001 C CNN
-F 1 "GND" H 3505 7427 50  0001 C CNN
-F 2 "" H 3500 7600 50  0001 C CNN
-F 3 "" H 3500 7600 50  0001 C CNN
-	1    3500 7600
-	1    0    0    -1
-$EndComp
-Wire Wire Line
-	3500 7550 3500 7600
-Wire Wire Line
-	3350 7550 3350 7600
+P 3600 7600
+F 0 "#PWR011" H 3600 7350 50  0001 C CNN
+F 1 "GND" H 3605 7427 50  0001 C CNN
+F 2 "" H 3600 7600 50  0001 C CNN
+F 3 "" H 3600 7600 50  0001 C CNN
+	1    3600 7600
+	1    0    0    -1
+$EndComp
+Wire Wire Line
+	3600 7550 3600 7600
+Wire Wire Line
+	3400 7550 3400 7600
 Wire Wire Line
 	3200 7550 3200 7600
@@
 L power:GND #PWR?
 U 1 1 61C91224
-P 3650 7600
-F 0 "#PWR?" H 3650 7350 50  0001 C CNN
-F 1 "GND" H 3655 7427 50  0001 C CNN
-F 2 "" H 3650 7600 50  0001 C CNN
-F 3 "" H 3650 7600 50  0001 C CNN
-	1    3650 7600
-	1    0    0    -1
-$EndComp
-Wire Wire Line
-	3650 7600 3650 7550
+P 3800 7600
+F 0 "#PWR?" H 3800 7350 50  0001 C CNN
+F 1 "GND" H 3805 7427 50  0001 C CNN
+F 2 "" H 3800 7600 50  0001 C CNN
+F 3 "" H 3800 7600 50  0001 C CNN
+	1    3800 7600
+	1    0    0    -1
+$EndComp
+Wire Wire Line
+	3800 7600 3800 7550
 Wire Wire Line
 	4650 6250 4650 6275
+$Comp
+L power:GND #PWR?
+U 1 1 61D533B7
+P 4000 7600
+F 0 "#PWR?" H 4000 7350 50  0001 C CNN
+F 1 "GND" H 4005 7427 50  0001 C CNN
+F 2 "" H 4000 7600 50  0001 C CNN
+F 3 "" H 4000 7600 50  0001 C CNN
+	1    4000 7600
+	1    0    0    -1
+$EndComp
+Wire Wire Line
+	4000 7550 4000 7600
 $EndSCHEMATC
